File: HardWare/EtherCAT2XXX.kicad_pcb (KiCad board)
At the start: 2 copper layers, 144 parts, among them CN1 5019530507, CN2 5019530507, J1 Conn_01x02, J2 Conn_01x03, J3 Conn_01x04, J4 Conn_01x02, J5 Conn_01x02, J6 Conn_01x03, J7 Conn_01x04, SW1 SW_Push, U1 SY8303AAIC, U2 RT8075, U3 SRV05-4, U4 SRV05-4, U5 STM32F407VETx, U6 TJA1051T-3, U7 TJA1051T-3, U8 AX58100-LQPF80, U9 BL24C16F-PARC, X1 25M, Y1 8M, Y2 32.768KHz

Commit message: First setting of firmware
Connections:
- U5 pad 15: unconnected-(U5-Pad15) -> /MCU/LED1
- U5 pad 23: /MCU/LED1 -> unconnected-(U5-Pad23)
- U5 pad 48: unconnected-(U5-Pad48) -> /MCU/LED3
- U5 pad 67: /MCU/LED3 -> unconnected-(U5-Pad67)
Changed lines of the file:
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@@
   (net 164 "/MCU/OSC32_IN")
   (net 165 "/MCU/OSC32_OUT")
-  (net 166 "unconnected-(U5-Pad15)")
+  (net 166 "unconnected-(U5-Pad23)")
   (net 167 "unconnected-(U5-Pad33)")
   (net 168 "unconnected-(U5-Pad34)")
@@
   (net 171 "unconnected-(U5-Pad45)")
   (net 172 "unconnected-(U5-Pad46)")
-  (net 173 "unconnected-(U5-Pad48)")
+  (net 173 "unconnected-(U5-Pad67)")
   (net 174 "unconnected-(U5-Pad55)")
   (net 175 "unconnected-(U5-Pad56)")
@@
       (net 150 "/MCU/RSET") (pinfunction "NRST") (pintype "input"))
     (pad "15" smd roundrect (at -7.675 1) (size 1.6 0.3) (layers "F.Cu" "F.Paste" "F.Mask") (roundrect_rratio 0.25)
-      (net 166 "unconnected-(U5-Pad15)") (pinfunction "PC0") (pintype "bidirectional+no_connect"))
+      (net 39 "/MCU/LED1") (pinfunction "PC0") (pintype "bidirectional"))
     (pad "16" smd roundrect (at -7.675 1.5) (size 1.6 0.3) (layers "F.Cu" "F.Paste" "F.Mask") (roundrect_rratio 0.25)
       (net 93 "/ESC/SYNC") (pinfunction "PC1") (pintype "bidirectional"))
@@
       (net 149 "/MCU/VREF") (pinfunction "VDDA") (pintype "power_in"))
     (pad "23" smd roundrect (at -7.675 5) (size 1.6 0.3) (layers "F.Cu" "F.Paste" "F.Mask") (roundrect_rratio 0.25)
-      (net 39 "/MCU/LED1") (pinfunction "PA0") (pintype "bidirectional"))
+      (net 166 "unconnected-(U5-Pad23)") (pinfunction "PA0") (pintype "bidirectional+no_connect"))
     (pad "24" smd roundrect (at -7.675 5.5) (size 1.6 0.3) (layers "F.Cu" "F.Paste" "F.Mask") (roundrect_rratio 0.25)
       (net 41 "/MCU/LED2") (pinfunction "PA1") (pintype "bidirectional"))
@@
       (net 157 "/MCU/SPI2_SCK") (pinfunction "PB10") (pintype "bidirectional"))
     (pad "48" smd roundrect (at 5 7.675) (size 0.3 1.6) (layers "F.Cu" "F.Paste" "F.Mask") (roundrect_rratio 0.25)
-      (net 173 "unconnected-(U5-Pad48)") (pinfunction "PB11") (pintype "bidirectional+no_connect"))
+      (net 43 "/MCU/LED3") (pinfunction "PB11") (pintype "bidirectional"))
     (pad "49" smd roundrect (at 5.5 7.675) (size 0.3 1.6) (layers "F.Cu" "F.Paste" "F.Mask") (roundrect_rratio 0.25)
       (net 147 "Net-(C50-Pad2)") (pinfunction "VCAP_1") (pintype "power_in"))
@@
       (net 185 "unconnected-(U5-Pad66)") (pinfunction "PC9") (pintype "bidirectional+no_connect"))
     (pad "67" smd roundrect (at 7.675 -2) (size 1.6 0.3) (layers "F.Cu" "F.Paste" "F.Mask") (roundrect_rratio 0.25)
-      (net 43 "/MCU/LED3") (pinfunction "PA8") (pintype "bidirectional"))
+      (net 173 "unconnected-(U5-Pad67)") (pinfunction "PA8") (pintype "bidirectional+no_connect"))
     (pad "68" smd roundrect (at 7.675 -2.5) (size 1.6 0.3) (layers "F.Cu" "F.Paste" "F.Mask") (roundrect_rratio 0.25)
       (net 152 "/MCU/USART1_TX") (pinfunction "PA9") (pintype "bidirectional"))
