File: HardWare/MCU.kicad_sch (KiCad schematic)
At the start: 40 parts, among them J2 Conn_01x03, J3 Conn_01x04, J6 Conn_01x03, J7 Conn_01x04, SW1 SW_Push, U5 STM32F407VETx, U6 TJA1051T-3, U7 TJA1051T-3, Y1 8M, Y2 32.768KHz

Commit message: First setting of firmware
Connections:
- net LED1: now also U5.15 (PC0); no longer U5.23 (PA0)
- net LED3: now also U5.48 (PB11); no longer U5.67 (PA8)
Changed lines of the file:
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@@
   (no_connect (at 110.49 88.9))
   (no_connect (at 110.49 81.28))
+  (no_connect (at 110.49 43.18))
   (no_connect (at 64.77 139.7))
   (no_connect (at 64.77 137.16))
@@
   (no_connect (at 64.77 144.78))
   (no_connect (at 64.77 142.24))
-  (no_connect (at 110.49 114.3))
-  (no_connect (at 110.49 129.54))
   (no_connect (at 110.49 139.7))
   (no_connect (at 110.49 142.24))
@@
   (no_connect (at 64.77 160.02))
   (no_connect (at 64.77 157.48))
+  (no_connect (at 110.49 63.5))
   (wire (pts (xy 192.024 39.116) (xy 199.644 39.116))
     (stroke (width 0) (type default) (color 0 0 0 0))
@@
     (effects (font (size 1.27 1.27)) (justify left bottom))
   )
-  (label "LED3" (at 110.49 63.5 0)
-    (effects (font (size 1.27 1.27)) (justify left bottom))
-  )
   (label "LED4" (at 250.19 70.358 0)
     (effects (font (size 1.27 1.27)) (justify left bottom))
@@
     (effects (font (size 1.27 1.27)) (justify left bottom))
   )
+  (label "LED1" (at 110.49 129.54 0)
+    (effects (font (size 1.27 1.27)) (justify left bottom))
+  )
   (label "SPI2_NSS" (at 110.49 109.22 0)
     (effects (font (size 1.27 1.27)) (justify left bottom))
@@
     (effects (font (size 1.27 1.27)) (justify right bottom))
   )
+  (label "LED3" (at 110.49 114.3 0)
+    (effects (font (size 1.27 1.27)) (justify left bottom))
+  )
   (label "USART2_RX" (at 110.49 50.8 0)
     (effects (font (size 1.27 1.27)) (justify left bottom))
@@
     (effects (font (size 1.27 1.27)) (justify left bottom))
   )
-  (label "LED1" (at 110.49 43.18 0)
-    (effects (font (size 1.27 1.27)) (justify left bottom))
-  )
