File: HardWare/ethercat_shield/CONN.kicad_sch (KiCad schematic)
At the start: 26 parts, among them CN1 5019530507, CN2 5019530507, J4 Conn_01x02, J5 Conn_01x02, U3 SRV05-4, U4 SRV05-4

Commit message: Add test version
Parts:
- added J8: USB_C_Receptacle_USB2.0, Connector_USB:USB_C_Receptacle_HRO_TYPE-C-31-M-12, symbol Connector:USB_C_Receptacle_USB2.0
Connections:
- net GNDA is gone; now on net GND: U3.2 (VN), U4.2 (VN)
- net Earth: now also J8.A1 (GND), J8.A12 (GND), J8.B1 (GND), J8.B12 (GND), J8.S1 (SHIELD)
- new net +5V: J8.A4 (VBUS), J8.A9 (VBUS), J8.B4 (VBUS), J8.B9 (VBUS)
- no-connect marks 4 -> 12
Other:
- moved on the sheet: C22, C23, C24, C25, L4, R12, R13, R14, R15
