File: HardWare/ethercat_shield/POWER.kicad_sch (KiCad schematic)
At the start: 34 parts, among them U1 SY8303AAIC, U2 RT8075

Commit message: Add test version
Parts:
- removed C1: 4.7u, Capacitor_SMD:C_0603_1608Metric, symbol Device:C
- removed C2, C3: 10n, Capacitor_SMD:C_0603_1608Metric, symbol Device:C
- removed C4: 22u, Capacitor_SMD:C_0603_1608Metric, symbol Device:C
- removed L1: 22uH, Inductor_SMD:L_6.3x6.3_H3, symbol Device:L
- removed R1: 100K, Resistor_SMD:R_0603_1608Metric, symbol Device:R
- removed R2: 150K, Resistor_SMD:R_0603_1608Metric, symbol Device:R
- removed R3: 20.5K, Resistor_SMD:R_0603_1608Metric, symbol Device:R
- removed U1: SY8303AAIC, EXTRA IC:SOT-23-8_L3.0-W1.7-P0.65-LS2.8-BR, symbol ECAT:SY8303AAIC
Connections:
- net GNDA is gone; now on net GND: C15.2, C16.2, C17.2, C18.2
- net GNDD is gone; now on net GND: C11.2, C12.2, C13.2, C14.2, R5.2, R7.2
