File: HardWare/ethercat_simple_test/POWER.kicad_sch (KiCad schematic)
At the start: 25 parts, among them U2 RT8075

Commit message: Pure test version
Parts:
- R4: value 453k -> 680k
- R5: value 100K -> 150K
- R6: value 453k -> 200k
- R7: value 100K -> 200K
