File: HardWare/ethercat/CONN.kicad_sch (KiCad schematic)
At the start: 26 parts, among them CN1 5019530507, CN2 5019530507, J4 Conn_01x02, J5 Conn_01x02, U3 SRV05-4, U4 SRV05-4

Commit message: Official version-EtherCAT2CAN_NUC
Parts:
- added J3: Conn_01x04, Connector_JST:JST_GH_SM04B-GHS-TB_1x04-1MP_P1.25mm_Horizontal, symbol Connector_Generic:Conn_01x04
- C22, C23, C24, C25: footprint Capacitor_SMD:C_0603_1608Metric -> Capacitor_SMD:C_0402_1005Metric
- D1, D2: value LED -> GREEN; footprint LED_SMD:LED_0603_1608Metric -> LED_SMD:LED_0402_1005Metric
- R12, R13, R14, R15: footprint Resistor_SMD:R_0603_1608Metric -> Resistor_SMD:R_0402_1005Metric
Connections:
- net GND: now also J3.4 (Pin_4)
- new net +5V: J3.1 (Pin_1)
- no-connect marks 4 -> 6
Other:
- moved on the sheet: C22, C23, C24, C25, L4, R12, R13, R14, R15
