File: HardWare/ethercat/EtherCAT2XXX.kicad_sch (KiCad schematic)
At the start: 5 parts, among them J1 Conn_01x02

Commit message: Official version-EtherCAT2CAN_NUC
Parts:
- removed J1: Conn_01x02, Connector_AMASS:AMASS_XT30UPB-M_1x02_P5.0mm_Vertical, symbol Connector_Generic:Conn_01x02
