File: HardWare/ethercat/POWER.kicad_sch (KiCad schematic)
At the start: 34 parts, among them U1 SY8303AAIC, U2 RT8075

Commit message: Official version-EtherCAT2CAN_NUC
Parts:
- removed C1: 4.7u, Capacitor_SMD:C_0603_1608Metric, symbol Device:C
- removed C2, C3: 10n, Capacitor_SMD:C_0603_1608Metric, symbol Device:C
- removed C4: 22u, Capacitor_SMD:C_0603_1608Metric, symbol Device:C
- removed L1: 22uH, Inductor_SMD:L_6.3x6.3_H3, symbol Device:L
- removed R1: 100K, Resistor_SMD:R_0603_1608Metric, symbol Device:R
- removed R2: 150K, Resistor_SMD:R_0603_1608Metric, symbol Device:R
- removed R3: 20.5K, Resistor_SMD:R_0603_1608Metric, symbol Device:R
- removed U1: SY8303AAIC, EXTRA IC:SOT-23-8_L3.0-W1.7-P0.65-LS2.8-BR, symbol ECAT:SY8303AAIC
- added D12, D6: BV05C, Diode_SMD:D_SOD-323, symbol Device:D_TVS
- added D5 (x2): RED, LED_SMD:LED_0402_1005Metric, symbol Device:LED
- added R24 (x2): 1K, Resistor_SMD:R_0402_1005Metric, symbol Device:R_Small
- C10, C13, C14, C17, C18, C6, C8, C9: footprint Capacitor_SMD:C_0603_1608Metric -> Capacitor_SMD:C_0402_1005Metric
- R4: value 453k -> 680k; footprint Resistor_SMD:R_0603_1608Metric -> Resistor_SMD:R_0402_1005Metric
- R5: value 100K -> 150K; footprint Resistor_SMD:R_0603_1608Metric -> Resistor_SMD:R_0402_1005Metric
- R6: value 453k -> 200k; footprint Resistor_SMD:R_0603_1608Metric -> Resistor_SMD:R_0402_1005Metric
- R7: value 100K -> 200K; footprint Resistor_SMD:R_0603_1608Metric -> Resistor_SMD:R_0402_1005Metric
Connections:
- net +5V: now also D12.2 (A2), D6.2 (A2)
- net 1V2: now also R24.2
- net 3V3: now also R24.2
- net GND: now also D12.1 (A1), D5.1 (K), D5.1 (K), D6.1 (A1)
- new net: D5.2 (A), R24.1 (x2)
